File: embroidery/embroidery.kicad_sch (KiCad schematic)
At the start: 4 parts, among them U1 4009, U2 4001, U3 4001, U4 4009

Commit message: super cool thing check this out
Parts:
- added unit 2 of U1
- added unit 2 of U2
- added unit 1 of U3
- added unit 1 of U4
Connections:
- net +1V1: now reaches U1.3, U2.2
- net +1V1: now also U3.2, U4.3
- net GND: now reaches U4.4
- net GND: now also U1.4
- new net: U3.1, U4.2
- new net: U2.5, U3.3
- new net: U1.5, U2.4, U2.6
